File: Kicad Project/Kicad Project.kicad_pcb (KiCad board)
At the start: 2 copper layers, 176 parts, among them SW1 RotaryEncoder_Switch

Commit message: schematic inital version no rot
Parts:
- added U1: nice_nano, nice-nano-kicad-master:nice_nano, B.Cu at (335.8, 95.2)
- moved D70 31.8 mm to (316.7, 95.2), turned to 90 degrees
Connections:
- D1 pad 1: unconnected-(D1-K-Pad1) -> /Row1
- D1 pad 2: unconnected-(D1-A-Pad2) -> Net-(D1-A)
- D10 pad 1: unconnected-(D10-K-Pad1) -> /Row7
- D10 pad 2: unconnected-(D10-A-Pad2) -> Net-(D10-A)
- D11 pad 1: unconnected-(D11-K-Pad1) -> /Row7
- D11 pad 2: unconnected-(D11-A-Pad2) -> Net-(D11-A)
- D12 pad 1: unconnected-(D12-K-Pad1) -> /Row7
- D12 pad 2: unconnected-(D12-A-Pad2) -> Net-(D12-A)
- D13 pad 1: unconnected-(D13-K-Pad1) -> /Row7
- D13 pad 2: unconnected-(D13-A-Pad2) -> Net-(D13-A)
- D14 pad 1: unconnected-(D14-K-Pad1) -> /Row2
- D14 pad 2: unconnected-(D14-A-Pad2) -> Net-(D14-A)
- D15 pad 1: unconnected-(D15-K-Pad1) -> /Row2
- D15 pad 2: unconnected-(D15-A-Pad2) -> Net-(D15-A)
- D16 pad 1: unconnected-(D16-K-Pad1) -> /Row2
- D16 pad 2: unconnected-(D16-A-Pad2) -> Net-(D16-A)
- D17 pad 1: unconnected-(D17-K-Pad1) -> /Row2
- D17 pad 2: unconnected-(D17-A-Pad2) -> Net-(D17-A)
- D18 pad 1: unconnected-(D18-K-Pad1) -> /Row2
- D18 pad 2: unconnected-(D18-A-Pad2) -> Net-(D18-A)
- D19 pad 1: unconnected-(D19-K-Pad1) -> /Row2
- D19 pad 2: unconnected-(D19-A-Pad2) -> Net-(D19-A)
- D2 pad 1: unconnected-(D2-K-Pad1) -> /Row1
- D2 pad 2: unconnected-(D2-A-Pad2) -> Net-(D2-A)
- D20 pad 1: unconnected-(D20-K-Pad1) -> /Row2
- D20 pad 2: unconnected-(D20-A-Pad2) -> Net-(D20-A)
- D21 pad 1: unconnected-(D21-K-Pad1) -> /Row2
- D21 pad 2: unconnected-(D21-A-Pad2) -> Net-(D21-A)
- D22 pad 1: unconnected-(D22-K-Pad1) -> /Row6
- D22 pad 2: unconnected-(D22-A-Pad2) -> Net-(D22-A)
- D23 pad 1: unconnected-(D23-K-Pad1) -> /Row6
- D23 pad 2: unconnected-(D23-A-Pad2) -> Net-(D23-A)
- D24 pad 1: unconnected-(D24-K-Pad1) -> /Row6
- D24 pad 2: unconnected-(D24-A-Pad2) -> Net-(D24-A)
- D25 pad 1: unconnected-(D25-K-Pad1) -> /Row6
- D25 pad 2: unconnected-(D25-A-Pad2) -> Net-(D25-A)
- D26 pad 1: unconnected-(D26-K-Pad1) -> /Row6
- D26 pad 2: unconnected-(D26-A-Pad2) -> Net-(D26-A)
- D27 pad 1: unconnected-(D27-K-Pad1) -> /Row3
- D27 pad 2: unconnected-(D27-A-Pad2) -> Net-(D27-A)
- D28 pad 1: unconnected-(D28-K-Pad1) -> /Row3
- D28 pad 2: unconnected-(D28-A-Pad2) -> Net-(D28-A)
- D29 pad 1: unconnected-(D29-K-Pad1) -> /Row3
- D29 pad 2: unconnected-(D29-A-Pad2) -> Net-(D29-A)
- D3 pad 1: unconnected-(D3-K-Pad1) -> /Row1
- D3 pad 2: unconnected-(D3-A-Pad2) -> Net-(D3-A)
- D30 pad 1: unconnected-(D30-K-Pad1) -> /Row3
- D30 pad 2: unconnected-(D30-A-Pad2) -> Net-(D30-A)
- D31 pad 1: unconnected-(D31-K-Pad1) -> /Row3
- D31 pad 2: unconnected-(D31-A-Pad2) -> Net-(D31-A)
- D32 pad 1: unconnected-(D32-K-Pad1) -> /Row3
- D32 pad 2: unconnected-(D32-A-Pad2) -> Net-(D32-A)
- D33 pad 1: unconnected-(D33-K-Pad1) -> /Row3
- D33 pad 2: unconnected-(D33-A-Pad2) -> Net-(D33-A)
- D34 pad 1: unconnected-(D34-K-Pad1) -> /Row9
- D34 pad 2: unconnected-(D34-A-Pad2) -> Net-(D34-A)
- D35 pad 1: unconnected-(D35-K-Pad1) -> /Row9
- D35 pad 2: unconnected-(D35-A-Pad2) -> Net-(D35-A)
- D36 pad 1: unconnected-(D36-K-Pad1) -> /Row9
- D36 pad 2: unconnected-(D36-A-Pad2) -> Net-(D36-A)
- D37 pad 1: unconnected-(D37-K-Pad1) -> /Row9
- D37 pad 2: unconnected-(D37-A-Pad2) -> Net-(D37-A)
- D38 pad 1: unconnected-(D38-K-Pad1) -> /Row9
- D38 pad 2: unconnected-(D38-A-Pad2) -> Net-(D38-A)
- D39 pad 1: unconnected-(D39-K-Pad1) -> /Row4
- D39 pad 2: unconnected-(D39-A-Pad2) -> Net-(D39-A)
- D4 pad 1: unconnected-(D4-K-Pad1) -> /Row1
- D4 pad 2: unconnected-(D4-A-Pad2) -> Net-(D4-A)
- D40 pad 1: unconnected-(D40-K-Pad1) -> /Row4
- D40 pad 2: unconnected-(D40-A-Pad2) -> Net-(D40-A)
- D41 pad 1: unconnected-(D41-K-Pad1) -> /Row4
- D41 pad 2: unconnected-(D41-A-Pad2) -> Net-(D41-A)
- D42 pad 1: unconnected-(D42-K-Pad1) -> /Row4
- D42 pad 2: unconnected-(D42-A-Pad2) -> Net-(D42-A)
- D43 pad 1: unconnected-(D43-K-Pad1) -> /Row4
- D43 pad 2: unconnected-(D43-A-Pad2) -> Net-(D43-A)
- D44 pad 1: unconnected-(D44-K-Pad1) -> /Row4
- D44 pad 2: unconnected-(D44-A-Pad2) -> Net-(D44-A)
- D45 pad 1: unconnected-(D45-K-Pad1) -> /Row10
- D45 pad 2: unconnected-(D45-A-Pad2) -> Net-(D45-A)
- D46 pad 1: unconnected-(D46-K-Pad1) -> /Row10
- D46 pad 2: unconnected-(D46-A-Pad2) -> Net-(D46-A)
- D47 pad 1: unconnected-(D47-K-Pad1) -> /Row10
- D47 pad 2: unconnected-(D47-A-Pad2) -> Net-(D47-A)
- D48 pad 1: unconnected-(D48-K-Pad1) -> /Row10
- D48 pad 2: unconnected-(D48-A-Pad2) -> Net-(D48-A)
- D49 pad 1: unconnected-(D49-K-Pad1) -> /Row10
- D49 pad 2: unconnected-(D49-A-Pad2) -> Net-(D49-A)
- D5 pad 1: unconnected-(D5-K-Pad1) -> /Row1
- D5 pad 2: unconnected-(D5-A-Pad2) -> Net-(D5-A)
- D50 pad 1: unconnected-(D50-K-Pad1) -> /Row5
- D50 pad 2: unconnected-(D50-A-Pad2) -> Net-(D50-A)
- D51 pad 1: unconnected-(D51-K-Pad1) -> /Row5
- D51 pad 2: unconnected-(D51-A-Pad2) -> Net-(D51-A)
- D52 pad 1: unconnected-(D52-K-Pad1) -> /Row5
- D52 pad 2: unconnected-(D52-A-Pad2) -> Net-(D52-A)
- D53 pad 1: unconnected-(D53-K-Pad1) -> /Row5
- D53 pad 2: unconnected-(D53-A-Pad2) -> Net-(D53-A)
- D54 pad 1: unconnected-(D54-K-Pad1) -> /Row5
- D54 pad 2: unconnected-(D54-A-Pad2) -> Net-(D54-A)
- D55 pad 1: unconnected-(D55-K-Pad1) -> /Row5
- D55 pad 2: unconnected-(D55-A-Pad2) -> Net-(D55-A)
- D56 pad 1: unconnected-(D56-K-Pad1) -> /Row5
- D56 pad 2: unconnected-(D56-A-Pad2) -> Net-(D56-A)
- D57 pad 1: unconnected-(D57-K-Pad1) -> /Row11
- D57 pad 2: unconnected-(D57-A-Pad2) -> Net-(D57-A)
- D58 pad 1: unconnected-(D58-K-Pad1) -> /Row11
- D58 pad 2: unconnected-(D58-A-Pad2) -> Net-(D58-A)
- D59 pad 1: unconnected-(D59-K-Pad1) -> /Row11
- D59 pad 2: unconnected-(D59-A-Pad2) -> Net-(D59-A)
- D6 pad 1: unconnected-(D6-K-Pad1) -> /Row1
- D6 pad 2: unconnected-(D6-A-Pad2) -> Net-(D6-A)
- D60 pad 1: unconnected-(D60-K-Pad1) -> /Row6
- D60 pad 2: unconnected-(D60-A-Pad2) -> Net-(D60-A)
- D61 pad 1: unconnected-(D61-K-Pad1) -> /Row6
- D61 pad 2: unconnected-(D61-A-Pad2) -> Net-(D61-A)
- D62 pad 1: unconnected-(D62-K-Pad1) -> /Row12
- D62 pad 2: unconnected-(D62-A-Pad2) -> Net-(D62-A)
- D63 pad 1: unconnected-(D63-K-Pad1) -> /Row12
- D63 pad 2: unconnected-(D63-A-Pad2) -> Net-(D63-A)
- D64 pad 1: unconnected-(D64-K-Pad1) -> /Row7
- D64 pad 2: unconnected-(D64-A-Pad2) -> Net-(D64-A)
- D65 pad 1: unconnected-(D65-K-Pad1) -> /Row7
- D65 pad 2: unconnected-(D65-A-Pad2) -> Net-(D65-A)
- D66 pad 1: unconnected-(D66-K-Pad1) -> /Row6
- D66 pad 2: unconnected-(D66-A-Pad2) -> Net-(D66-A)
- D67 pad 1: unconnected-(D67-K-Pad1) -> /Row6
- D67 pad 2: unconnected-(D67-A-Pad2) -> Net-(D67-A)
- D68 pad 1: unconnected-(D68-K-Pad1) -> /Row9
- D68 pad 2: unconnected-(D68-A-Pad2) -> Net-(D68-A)
- D69 pad 1: unconnected-(D69-K-Pad1) -> /Row9
- D69 pad 2: unconnected-(D69-A-Pad2) -> Net-(D69-A)
- D7 pad 1: unconnected-(D7-K-Pad1) -> /Row1
- D7 pad 2: unconnected-(D7-A-Pad2) -> Net-(D7-A)
- D70 pad 1: unconnected-(D70-K-Pad1) -> /Row10
- D70 pad 2: unconnected-(D70-A-Pad2) -> Net-(D70-A)
- D71 pad 1: unconnected-(D71-K-Pad1) -> /Row11
- D71 pad 2: unconnected-(D71-A-Pad2) -> Net-(D71-A)
- D72 pad 1: unconnected-(D72-K-Pad1) -> /Row11
- D72 pad 2: unconnected-(D72-A-Pad2) -> Net-(D72-A)
- D73 pad 1: unconnected-(D73-K-Pad1) -> /Row12
- D73 pad 2: unconnected-(D73-A-Pad2) -> Net-(D73-A)
- D74 pad 1: unconnected-(D74-K-Pad1) -> /Row12
- D74 pad 2: unconnected-(D74-A-Pad2) -> Net-(D74-A)
- D75 pad 1: unconnected-(D75-K-Pad1) -> /Row12
- D75 pad 2: unconnected-(D75-A-Pad2) -> Net-(D75-A)
- D76 pad 1: unconnected-(D76-K-Pad1) -> /Row6
- D76 pad 2: unconnected-(D76-A-Pad2) -> Net-(D76-A)
- D77 pad 1: unconnected-(D77-K-Pad1) -> /Row6
- D77 pad 2: unconnected-(D77-A-Pad2) -> Net-(D77-A)
- D78 pad 1: unconnected-(D78-K-Pad1) -> /Row12
- D78 pad 2: unconnected-(D78-A-Pad2) -> Net-(D78-A)
- D79 pad 1: unconnected-(D79-K-Pad1) -> /Row3
- D79 pad 2: unconnected-(D79-A-Pad2) -> Net-(D79-A)
- D8 pad 1: unconnected-(D8-K-Pad1) -> /Row1
- D8 pad 2: unconnected-(D8-A-Pad2) -> Net-(D8-A)
- D80 pad 1: unconnected-(D80-K-Pad1) -> /Row9
- D80 pad 2: unconnected-(D80-A-Pad2) -> Net-(D80-A)
- D81 pad 1: unconnected-(D81-K-Pad1) -> /Row4
- D81 pad 2: unconnected-(D81-A-Pad2) -> Net-(D81-A)
- D82 pad 1: unconnected-(D82-K-Pad1) -> /Row6
- D82 pad 2: unconnected-(D82-A-Pad2) -> Net-(D82-A)
- D83 pad 1: unconnected-(D83-K-Pad1) -> /Row10
- D83 pad 2: unconnected-(D83-A-Pad2) -> Net-(D83-A)
- D84 pad 1: unconnected-(D84-K-Pad1) -> /Row5
- D84 pad 2: unconnected-(D84-A-Pad2) -> Net-(D84-A)
- D85 pad 1: unconnected-(D85-K-Pad1) -> /Row11
- D85 pad 2: unconnected-(D85-A-Pad2) -> Net-(D85-A)
- D86 pad 1: unconnected-(D86-K-Pad1) -> /Row6
- D86 pad 2: unconnected-(D86-A-Pad2) -> Net-(D86-A)
- D87 pad 1: unconnected-(D87-K-Pad1) -> /Row7
- D87 pad 2: unconnected-(D87-A-Pad2) -> /RSw2
- D9 pad 1: unconnected-(D9-K-Pad1) -> /Row7
- D9 pad 2: unconnected-(D9-A-Pad2) -> Net-(D9-A)
- MX1 pad 1: unconnected-(MX1-COL-Pad1) -> /Col1
- MX1 pad 2: unconnected-(MX1-ROW-Pad2) -> Net-(D1-A)
- MX10 pad 1: unconnected-(MX10-COL-Pad1) -> /Col7
- MX10 pad 2: unconnected-(MX10-ROW-Pad2) -> Net-(D10-A)
- MX11 pad 1: unconnected-(MX11-COL-Pad1) -> /Col3
- MX11 pad 2: unconnected-(MX11-ROW-Pad2) -> Net-(D11-A)
- MX12 pad 1: unconnected-(MX12-COL-Pad1) -> /Col6
- MX12 pad 2: unconnected-(MX12-ROW-Pad2) -> Net-(D12-A)
- MX13 pad 1: unconnected-(MX13-COL-Pad1) -> /Col5
- MX13 pad 2: unconnected-(MX13-ROW-Pad2) -> Net-(D13-A)
- MX14 pad 1: unconnected-(MX14-COL-Pad1) -> /Col1
- MX14 pad 2: unconnected-(MX14-ROW-Pad2) -> Net-(D14-A)
- MX15 pad 1: unconnected-(MX15-COL-Pad1) -> /Col2
- MX15 pad 2: unconnected-(MX15-ROW-Pad2) -> Net-(D15-A)
- MX16 pad 1: unconnected-(MX16-COL-Pad1) -> /Col3
- MX16 pad 2: unconnected-(MX16-ROW-Pad2) -> Net-(D16-A)
- MX17 pad 1: unconnected-(MX17-COL-Pad1) -> /Col4
- MX17 pad 2: unconnected-(MX17-ROW-Pad2) -> Net-(D17-A)
- MX18 pad 1: unconnected-(MX18-COL-Pad1) -> /Col5
- MX18 pad 2: unconnected-(MX18-ROW-Pad2) -> Net-(D18-A)
- MX19 pad 1: unconnected-(MX19-COL-Pad1) -> /Col6
- MX19 pad 2: unconnected-(MX19-ROW-Pad2) -> Net-(D19-A)
- MX2 pad 1: unconnected-(MX2-COL-Pad1) -> /Col2
- MX2 pad 2: unconnected-(MX2-ROW-Pad2) -> Net-(D2-A)
- MX20 pad 1: unconnected-(MX20-COL-Pad1) -> /Col7
- MX20 pad 2: unconnected-(MX20-ROW-Pad2) -> Net-(D20-A)
- MX21 pad 1: unconnected-(MX21-COL-Pad1) -> /Col8
- MX21 pad 2: unconnected-(MX21-ROW-Pad2) -> Net-(D21-A)
- MX22 pad 1: unconnected-(MX22-COL-Pad1) -> /Col8
- MX22 pad 2: unconnected-(MX22-ROW-Pad2) -> Net-(D22-A)
- MX23 pad 1: unconnected-(MX23-COL-Pad1) -> /Col7
- MX23 pad 2: unconnected-(MX23-ROW-Pad2) -> Net-(D23-A)
- MX24 pad 1: unconnected-(MX24-COL-Pad1) -> /Col6
- MX24 pad 2: unconnected-(MX24-ROW-Pad2) -> Net-(D24-A)
- MX25 pad 1: unconnected-(MX25-COL-Pad1) -> /Col5
- MX25 pad 2: unconnected-(MX25-ROW-Pad2) -> Net-(D25-A)
- MX26 pad 1: unconnected-(MX26-COL-Pad1) -> /Col4
- MX26 pad 2: unconnected-(MX26-ROW-Pad2) -> Net-(D26-A)
- MX27 pad 1: unconnected-(MX27-COL-Pad1) -> /Col2
- MX27 pad 2: unconnected-(MX27-ROW-Pad2) -> Net-(D27-A)
- MX28 pad 1: unconnected-(MX28-COL-Pad1) -> /Col3
- MX28 pad 2: unconnected-(MX28-ROW-Pad2) -> Net-(D28-A)
- MX29 pad 1: unconnected-(MX29-COL-Pad1) -> /Col4
- MX29 pad 2: unconnected-(MX29-ROW-Pad2) -> Net-(D29-A)
- MX3 pad 1: unconnected-(MX3-COL-Pad1) -> /Col3
- MX3 pad 2: unconnected-(MX3-ROW-Pad2) -> Net-(D3-A)
- MX30 pad 1: unconnected-(MX30-COL-Pad1) -> /Col5
- MX30 pad 2: unconnected-(MX30-ROW-Pad2) -> Net-(D30-A)
- MX31 pad 1: unconnected-(MX31-COL-Pad1) -> /Col6
- MX31 pad 2: unconnected-(MX31-ROW-Pad2) -> Net-(D31-A)
- MX32 pad 1: unconnected-(MX32-COL-Pad1) -> /Col7
- MX32 pad 2: unconnected-(MX32-ROW-Pad2) -> Net-(D32-A)
- MX33 pad 1: unconnected-(MX33-COL-Pad1) -> /Col8
- MX33 pad 2: unconnected-(MX33-ROW-Pad2) -> Net-(D33-A)
- MX34 pad 1: unconnected-(MX34-COL-Pad1) -> /Col8
- MX34 pad 2: unconnected-(MX34-ROW-Pad2) -> Net-(D34-A)
- MX35 pad 1: unconnected-(MX35-COL-Pad1) -> /Col7
- MX35 pad 2: unconnected-(MX35-ROW-Pad2) -> Net-(D35-A)
- MX36 pad 1: unconnected-(MX36-COL-Pad1) -> /Col6
- MX36 pad 2: unconnected-(MX36-ROW-Pad2) -> Net-(D36-A)
- MX37 pad 1: unconnected-(MX37-COL-Pad1) -> /Col5
- MX37 pad 2: unconnected-(MX37-ROW-Pad2) -> Net-(D37-A)
- MX38 pad 1: unconnected-(MX38-COL-Pad1) -> /Col4
- MX38 pad 2: unconnected-(MX38-ROW-Pad2) -> Net-(D38-A)
- MX39 pad 1: unconnected-(MX39-COL-Pad1) -> /Col2
- MX39 pad 2: unconnected-(MX39-ROW-Pad2) -> Net-(D39-A)
- MX4 pad 1: unconnected-(MX4-COL-Pad1) -> /Col4
- MX4 pad 2: unconnected-(MX4-ROW-Pad2) -> Net-(D4-A)
- MX40 pad 1: unconnected-(MX40-COL-Pad1) -> /Col3
- MX40 pad 2: unconnected-(MX40-ROW-Pad2) -> Net-(D40-A)
- MX41 pad 1: unconnected-(MX41-COL-Pad1) -> /Col4
- MX41 pad 2: unconnected-(MX41-ROW-Pad2) -> Net-(D41-A)
- MX42 pad 1: unconnected-(MX42-COL-Pad1) -> /Col5
- MX42 pad 2: unconnected-(MX42-ROW-Pad2) -> Net-(D42-A)
- MX43 pad 1: unconnected-(MX43-COL-Pad1) -> /Col6
- MX43 pad 2: unconnected-(MX43-ROW-Pad2) -> Net-(D43-A)
- MX44 pad 1: unconnected-(MX44-COL-Pad1) -> /Col7
- MX44 pad 2: unconnected-(MX44-ROW-Pad2) -> Net-(D44-A)
- MX45 pad 1: unconnected-(MX45-COL-Pad1) -> /Col8
- MX45 pad 2: unconnected-(MX45-ROW-Pad2) -> Net-(D45-A)
- MX46 pad 1: unconnected-(MX46-COL-Pad1) -> /Col7
- MX46 pad 2: unconnected-(MX46-ROW-Pad2) -> Net-(D46-A)
- MX47 pad 1: unconnected-(MX47-COL-Pad1) -> /Col6
- MX47 pad 2: unconnected-(MX47-ROW-Pad2) -> Net-(D47-A)
- MX48 pad 1: unconnected-(MX48-COL-Pad1) -> /Col5
- MX48 pad 2: unconnected-(MX48-ROW-Pad2) -> Net-(D48-A)
- MX49 pad 1: unconnected-(MX49-COL-Pad1) -> /Col4
- MX49 pad 2: unconnected-(MX49-ROW-Pad2) -> Net-(D49-A)
- MX5 pad 1: unconnected-(MX5-COL-Pad1) -> /Col5
- MX5 pad 2: unconnected-(MX5-ROW-Pad2) -> Net-(D5-A)
- MX50 pad 1: unconnected-(MX50-COL-Pad1) -> /Col2
- MX50 pad 2: unconnected-(MX50-ROW-Pad2) -> Net-(D50-A)
- MX51 pad 1: unconnected-(MX51-COL-Pad1) -> /Col3
- MX51 pad 2: unconnected-(MX51-ROW-Pad2) -> Net-(D51-A)
- MX52 pad 1: unconnected-(MX52-COL-Pad1) -> /Col4
- MX52 pad 2: unconnected-(MX52-ROW-Pad2) -> Net-(D52-A)
- MX53 pad 1: unconnected-(MX53-COL-Pad1) -> /Col5
- MX53 pad 2: unconnected-(MX53-ROW-Pad2) -> Net-(D53-A)
- MX54 pad 1: unconnected-(MX54-COL-Pad1) -> /Col6
- MX54 pad 2: unconnected-(MX54-ROW-Pad2) -> Net-(D54-A)
- MX55 pad 1: unconnected-(MX55-COL-Pad1) -> /Col7
- MX55 pad 2: unconnected-(MX55-ROW-Pad2) -> Net-(D55-A)
- MX56 pad 1: unconnected-(MX56-COL-Pad1) -> /Col8
- MX56 pad 2: unconnected-(MX56-ROW-Pad2) -> Net-(D56-A)
- MX57 pad 1: unconnected-(MX57-COL-Pad1) -> /Col6
- MX57 pad 2: unconnected-(MX57-ROW-Pad2) -> Net-(D57-A)
- MX58 pad 1: unconnected-(MX58-COL-Pad1) -> /Col5
- MX58 pad 2: unconnected-(MX58-ROW-Pad2) -> Net-(D58-A)
- MX59 pad 1: unconnected-(MX59-COL-Pad1) -> /Col4
- MX59 pad 2: unconnected-(MX59-ROW-Pad2) -> Net-(D59-A)
- MX6 pad 1: unconnected-(MX6-COL-Pad1) -> /Col6
- MX6 pad 2: unconnected-(MX6-ROW-Pad2) -> Net-(D6-A)
- MX60 pad 1: unconnected-(MX60-COL-Pad1) -> /Col2
- MX60 pad 2: unconnected-(MX60-ROW-Pad2) -> Net-(D60-A)
- MX61 pad 1: unconnected-(MX61-COL-Pad1) -> /Col3
- MX61 pad 2: unconnected-(MX61-ROW-Pad2) -> Net-(D61-A)
- MX62 pad 1: unconnected-(MX62-COL-Pad1) -> /Col6
- MX62 pad 2: unconnected-(MX62-ROW-Pad2) -> Net-(D62-A)
- MX63 pad 1: unconnected-(MX63-COL-Pad1) -> /Col5
- MX63 pad 2: unconnected-(MX63-ROW-Pad2) -> Net-(D63-A)
- MX64 pad 1: unconnected-(MX64-COL-Pad1) -> /Col4
- MX64 pad 2: unconnected-(MX64-ROW-Pad2) -> Net-(D64-A)
- MX65 pad 1: unconnected-(MX65-COL-Pad1) -> /Col2
- MX65 pad 2: unconnected-(MX65-ROW-Pad2) -> Net-(D65-A)
- MX66 pad 1: unconnected-(MX66-COL-Pad1) -> /Col2
- MX66 pad 2: unconnected-(MX66-ROW-Pad2) -> Net-(D66-A)
- MX67 pad 1: unconnected-(MX67-COL-Pad1) -> /Col1
- MX67 pad 2: unconnected-(MX67-ROW-Pad2) -> Net-(D67-A)
- MX68 pad 1: unconnected-(MX68-COL-Pad1) -> /Col2
- MX68 pad 2: unconnected-(MX68-ROW-Pad2) -> Net-(D68-A)
- MX69 pad 1: unconnected-(MX69-COL-Pad1) -> /Col1
- MX69 pad 2: unconnected-(MX69-ROW-Pad2) -> Net-(D69-A)
- MX7 pad 1: unconnected-(MX7-COL-Pad1) -> /Col7
- MX7 pad 2: unconnected-(MX7-ROW-Pad2) -> Net-(D7-A)
- MX70 pad 1: unconnected-(MX70-COL-Pad1) -> /Col1
- MX70 pad 2: unconnected-(MX70-ROW-Pad2) -> Net-(D70-A)
- MX71 pad 1: unconnected-(MX71-COL-Pad1) -> /Col1
- MX71 pad 2: unconnected-(MX71-ROW-Pad2) -> Net-(D71-A)
- MX72 pad 1: unconnected-(MX72-COL-Pad1) -> /Col2
- MX72 pad 2: unconnected-(MX72-ROW-Pad2) -> Net-(D72-A)
- MX73 pad 1: unconnected-(MX73-COL-Pad1) -> /Col3
- MX73 pad 2: unconnected-(MX73-ROW-Pad2) -> Net-(D73-A)
- MX74 pad 1: unconnected-(MX74-COL-Pad1) -> /Col2
- MX74 pad 2: unconnected-(MX74-ROW-Pad2) -> Net-(D74-A)
- MX75 pad 1: unconnected-(MX75-COL-Pad1) -> /Col1
- MX75 pad 2: unconnected-(MX75-ROW-Pad2) -> Net-(D75-A)
- MX76 pad 1: unconnected-(MX76-COL-Pad1) -> /Col1
- MX76 pad 2: unconnected-(MX76-ROW-Pad2) -> Net-(D76-A)
- MX77 pad 1: unconnected-(MX77-COL-Pad1) -> /Col4
- MX77 pad 2: unconnected-(MX77-ROW-Pad2) -> Net-(D77-A)
- MX78 pad 1: unconnected-(MX78-COL-Pad1) -> /Col4
- MX78 pad 2: unconnected-(MX78-ROW-Pad2) -> Net-(D78-A)
- MX79 pad 1: unconnected-(MX79-COL-Pad1) -> /Col1
- MX79 pad 2: unconnected-(MX79-ROW-Pad2) -> Net-(D79-A)
- MX8 pad 1: unconnected-(MX8-COL-Pad1) -> /Col8
- MX8 pad 2: unconnected-(MX8-ROW-Pad2) -> Net-(D8-A)
- MX80 pad 1: unconnected-(MX80-COL-Pad1) -> /Col3
- MX80 pad 2: unconnected-(MX80-ROW-Pad2) -> Net-(D80-A)
- MX81 pad 1: unconnected-(MX81-COL-Pad1) -> /Col1
- MX81 pad 2: unconnected-(MX81-ROW-Pad2) -> Net-(D81-A)
- MX82 pad 1: unconnected-(MX82-COL-Pad1) -> /Col3
- MX82 pad 2: unconnected-(MX82-ROW-Pad2) -> Net-(D82-A)
- MX83 pad 1: unconnected-(MX83-COL-Pad1) -> /Col3
- MX83 pad 2: unconnected-(MX83-ROW-Pad2) -> Net-(D83-A)
- MX84 pad 1: unconnected-(MX84-COL-Pad1) -> /Col1
- MX84 pad 2: unconnected-(MX84-ROW-Pad2) -> Net-(D84-A)
- MX85 pad 1: unconnected-(MX85-COL-Pad1) -> /Col3
- MX85 pad 2: unconnected-(MX85-ROW-Pad2) -> Net-(D85-A)
- MX86 pad 1: unconnected-(MX86-COL-Pad1) -> /Col5
- MX86 pad 2: unconnected-(MX86-ROW-Pad2) -> Net-(D86-A)
- MX9 pad 1: unconnected-(MX9-COL-Pad1) -> /Col8
- MX9 pad 2: unconnected-(MX9-ROW-Pad2) -> Net-(D9-A)
- SW1 pad A: unconnected-(SW1-PadA) -> /RRotA
- SW1 pad B: unconnected-(SW1-PadB) -> /RRotC
- SW1 pad C: unconnected-(SW1-PadC) -> /RRotB
- SW1 pad S1: unconnected-(SW1-PadS1) -> /Col1
- SW1 pad S2: unconnected-(SW1-PadS2) -> /RSw2
Other:
- board outline added: 342.9 x 126.2 mm

Commit message: routed minus rot and controller
Parts:
- removed D89: 1N4148W, Diode_SMD:D_SOD-123
- moved D11 7.14 mm to (235.7, 45.2), turned to 90 degrees
- moved D13 7.14 mm to (273.8, 45.2), turned to 90 degrees
- moved D19 7.14 mm to (140.5, 64.3), turned to 90 degrees
- moved D21 7.14 mm to (178.6, 64.3), turned to 90 degrees
- moved D22 7.14 mm to (197.6, 64.3), turned to 90 degrees
- moved D24 7.14 mm to (235.7, 64.3), turned to 90 degrees
- moved D26 7.14 mm to (273.8, 64.3), turned to 90 degrees
- moved D28 7.14 mm to (92.9, 83.3), turned to 90 degrees
- moved D31 7.14 mm to (150.0, 83.3), turned to 90 degrees
- moved D33 7.14 mm to (188.1, 83.3), turned to 90 degrees
- moved D35 7.14 mm to (226.2, 83.3), turned to 90 degrees
- moved D36 7.14 mm to (245.3, 83.3), turned to 90 degrees
- moved D37 7.14 mm to (264.3, 83.3), turned to 90 degrees
- moved D41 7.14 mm to (116.7, 102.4), turned to 90 degrees
- moved D43 7.14 mm to (154.8, 102.4), turned to 90 degrees
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Connections:
- D88 pad 1: unconnected-(D88-K-Pad1) -> /Row11
- D88 pad 2: unconnected-(D88-A-Pad2) -> /RRotC
- MX11 pad 1: /Col3 -> /Col6
- MX12 pad 1: /Col6 -> /Col5
- MX13 pad 1: /Col5 -> /Col4
- MX64 pad 1: /Col4 -> /Col3
- SW1 pad A: /RRotA -> /Col7
- SW1 pad B: /RRotC -> /Col7
- SW1 pad C: /RRotB -> /RRotC
Routing:
- net /Col1: track 0.00 -> 524.2 mm
- net /Col2: track 0.00 -> 497.9 mm
- net /Col3: track 0.00 -> 446.9 mm
- net /Col4: track 0.00 -> 393.3 mm
- net /Col5: track 0.00 -> 362.2 mm
- net /Col6: track 0.00 -> 315.6 mm
- net /Col7: track 0.00 -> 216.3 mm
- net /Row7: track 0.00 -> 157.2 mm
- net /Row5: track 0.00 -> 147.6 mm
- net /Row3: track 0.00 -> 138.1 mm
- net /Row6: track 0.00 -> 135.7 mm
- net /Col8: track 0.00 -> 135.3 mm
- net /Row2: track 0.00 -> 133.3 mm
- net /Row1: track 0.00 -> 133.3 mm
- net /Row4: track 0.00 -> 121.4 mm
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
Commit message: fully routed draft
Parts:
- moved D70 38.8 mm to (354.8, 102.4)
- moved D88 8.59 mm to (338.1, 50.0), turned to 0 degrees
Connections:
- D22 pad 1: /Row6 -> /Row8
- D23 pad 1: /Row6 -> /Row8
- D24 pad 1: /Row6 -> /Row8
- D25 pad 1: /Row6 -> /Row8
- D26 pad 1: /Row6 -> /Row8
- D66 pad 1: /Row6 -> /Row8
- D67 pad 1: /Row6 -> /Row8
- D82 pad 1: /Row6 -> /Row8
- SW1 pad B: /Col7 -> /Col8
- U1 pad 10: unconnected-(U1-P0.11-Pad10) -> /Row4
- U1 pad 11: unconnected-(U1-P1.04-Pad11) -> /Row5
- U1 pad 12: unconnected-(U1-P1.06-Pad12) -> /Row6
- U1 pad 13: unconnected-(U1-NFC1/P0.09-Pad13) -> /Row1
- U1 pad 14: unconnected-(U1-NFC2/P0.10-Pad14) -> /Row2
- U1 pad 15: unconnected-(U1-P1.11-Pad15) -> /Row3
- U1 pad 16: unconnected-(U1-P1.13-Pad16) -> /Col2
- U1 pad 17: unconnected-(U1-P1.15-Pad17) -> /Col1
- U1 pad 18: unconnected-(U1-AIN0/P0.02-Pad18) -> /Row7
- U1 pad 19: unconnected-(U1-AIN5/P0.29-Pad19) -> /Row8
- U1 pad 20: unconnected-(U1-AIN7/P0.31-Pad20) -> /Row9
- U1 pad 31: unconnected-(U1-P1.01-Pad31) -> /Col3
- U1 pad 32: unconnected-(U1-P1.02-Pad32) -> /Col8
- U1 pad 33: unconnected-(U1-P1.07-Pad33) -> /Col7
- U1 pad 5: unconnected-(U1-P0.17-Pad5) -> /Row11
- U1 pad 6: unconnected-(U1-P0.20-Pad6) -> /Row12
- U1 pad 7: unconnected-(U1-P0.22-Pad7) -> /Col4
- U1 pad 8: unconnected-(U1-P0.24-Pad8) -> /Col5
- U1 pad 9: unconnected-(U1-P1.00-Pad9) -> /Col6
Routing:
- net /Col8: track 135.3 -> 529.3 mm, vias 0 -> 1
- net /Col7: track 216.3 -> 579.2 mm, vias 0 -> 1
- net /Row11: track 0.00 -> 273.1 mm, vias 0 -> 4
- net /Col5: track 362.2 -> 582.1 mm, vias 0 -> 1
- net /Row8: track 0.00 -> 208.9 mm
- net /Col6: track 315.6 -> 520.9 mm, vias 0 -> 1
- net /Row6: track 135.7 -> 337.8 mm
- net /Col4: track 393.3 -> 576.9 mm, vias 0 -> 1
- net /Row5: track 147.6 -> 320.5 mm
- net /Row1: track 133.3 -> 305.7 mm
- net /Row12: track 0.00 -> 171.4 mm
- net /Row10: track 0.00 -> 170.5 mm
- net /Row2: track 133.3 -> 292.9 mm
- net /Row4: track 121.4 -> 278.5 mm
- net /Row9: track 0.00 -> 152.5 mm
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
Commit message: most diodes rerouted to back
Parts:
- added M3-1: MountingHole_3.2mm_M3, MountingHole:MountingHole_3.2mm_M3, F.Cu at (159.1, 168.7)
- added M3-2: MountingHole_3.2mm_M3, MountingHole:MountingHole_3.2mm_M3, F.Cu at (229.1, 168.7)
- D1, D10, D11, D12, D13, D14, D15, D16, D17, D18, D19, D2, D20, D21, D22, D23, D24, D25, D26, D27, D28, D29, D3, D30, D31, D32, D33, D34, D35, D36, D37, D38, D39, D4, D40, D41, D42, D43, D44, D45, D46, D47, D48, D49, D5, D6, D60, D61, D62, D63, D64, D65, D66, D67, D68, D69, D7, D70, D73, D74, D75, D76, D77, D78, D79, D8, D80, D81, D82, D83, D86, D87, D9: moved to B.Cu
- moved MX59 40.5 mm to (271.5, 150.0)
- moved D58 40.5 mm to (259.6, 157.2)
- moved D70 40.5 mm to (373.9, 138.1)
- moved MX50 40.5 mm to (100.0, 150.0)
- moved MX51 40.5 mm to (119.1, 150.0)
- moved MX52 40.5 mm to (138.1, 150.0)
- moved MX54 40.5 mm to (176.2, 150.0)
- moved MX55 40.5 mm to (195.3, 150.0)
- moved MX56 40.5 mm to (214.3, 150.0)
- moved MX57 40.5 mm to (233.4, 150.0)
- moved MX71 40.5 mm to (366.7, 150.0)
- moved MX72 40.5 mm to (347.7, 150.0)
- moved MX84 40.5 mm to (69.1, 150.0)
- moved MX85 40.5 mm to (307.2, 150.0)
- moved D51 40.5 mm to (126.2, 157.2)
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Connections:
- U1 pad 1: unconnected-(U1-TX0/P0.06-Pad1) -> /Col6
- U1 pad 32: /Col8 -> /Col7
- U1 pad 33: /Col7 -> /Col8
- U1 pad 5: /Row11 -> /Col5
- U1 pad 6: /Row12 -> /Col4
- U1 pad 7: /Col4 -> /Row12
- U1 pad 8: /Col5 -> /Row11
- U1 pad 9: /Col6 -> /Row10
Routing:
- net /Col6: track 520.9 -> 496.2 mm
- net /Col5: track 582.1 -> 569.0 mm
- net /Row1: track 305.7 -> 318.1 mm, vias 0 -> 14
- net /Col4: track 576.9 -> 568.9 mm
- net /Col8: track 529.3 -> 524.7 mm
- net /Row11: track 273.1 -> 276.2 mm
- net /Row9: track 152.5 -> 149.7 mm, vias 0 -> 10
- net /Row8: track 208.9 -> 206.3 mm, vias 0 -> 15
- net /Col1: track 546.8 -> 544.4 mm
- net /Col7: track 579.2 -> 576.8 mm
- net /Col3: track 521.6 -> 519.4 mm
- net /Col2: track 507.2 -> 505.1 mm
- net /Row7: track 228.3 -> 226.2 mm, vias 0 -> 15
- net /Row12: track 171.4 -> 169.5 mm, vias 0 -> 5
- net /Row4: track 278.5 -> 277.2 mm, vias 0 -> 15
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- added copper zone on B.Cu, net (none)
- added copper zone on F.Cu, net (none)
Other:
- board size 342.9 x 126.2 mm -> 336 x 122 mm
- board text added: "122"
- board text added: "14"
- board text added: "17"
- board text added: "336"
- board text added: "53"

Commit message: stable before rewire
Routing:
- net /Row5: track 320.3 -> 289.2 mm
- net /Row6: track 337.0 -> 306.0 mm

Commit message: pcbs ordered july 13th 2025
Parts:
- D50, D51, D52, D53, D54, D55, D56, D57, D58, D59, D71, D72, D84, D85, D88: moved to B.Cu
- turned D88 to 180 degrees
Connections:
- U1 pad 32: /Col7 -> /Col5
- U1 pad 5: /Col5 -> /Col7
Routing:
- net /Col2: track 505.1 -> 588.1 mm, vias 2 -> 5
- net /Col1: track 544.4 -> 614.3 mm, vias 0 -> 4
- net /Row11: track 276.2 -> 215.2 mm, vias 4 -> 1
- net /Col8: track 524.7 -> 486.1 mm, vias 1 -> 5
- net /Col7: track 576.8 -> 538.9 mm, vias 1 -> 9
- net /Col5: track 569.0 -> 535.7 mm, vias 1 -> 12
- net /Col3: track 519.4 -> 551.9 mm, vias 0 -> 12
- net /Col4: track 568.9 -> 544.3 mm, vias 1 -> 12
- net /Row12: track 169.5 -> 146.2 mm, vias 5 -> 1
- net /Row8: track 206.3 -> 183.5 mm, vias 15 -> 1
- net /Row7: track 226.2 -> 205.3 mm, vias 15 -> 1
- net /Col6: track 496.2 -> 512.6 mm, vias 1 -> 11
- net /Row1: track 318.1 -> 302.8 mm, vias 14 -> 0
- net /Row4: track 277.2 -> 283.9 mm, vias 15 -> 0
- net /Row6: track 306.0 -> 301.7 mm, vias 1 -> 0
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