File: Kicad Project/Kicad Project.kicad_sch (KiCad schematic)
At the start: 176 parts, among them SW1 RotaryEncoder_Switch

Commit message: schematic inital version no rot
Parts:
- added U1: nice_nano, nice-nano-kicad-master:nice_nano, symbol nice_nano:nice_nano
- D1, D10, D11, D12, D13, D14, D15, D16, D17, D18, D19, D2, D20, D21, D22, D23, D24, D25, D26, D27, D28, D29, D3, D30, D31, D32, D33, D34, D35, D36, D37, D38, D39, D4, D40, D41, D42, D43, D44, D45, D46, D47, D48, D49, D5, D50, D51, D52, D53, D54, D55, D56, D57, D58, D59, D6, D60, D61, D62, D63, D64, D65, D66, D67, D68, D69, D7, D70, D71, D72, D73, D74, D75, D76, D77, D78, D79, D8, D80, D81, D82, D83, D84, D85, D86, D87, D88, D89, D9: symbol Diode:1N4148W -> Device:D_Small
Connections:
- net Row12: now reaches D73.1 (K)
- net Row12: now also D62.1 (K), D63.1 (K), D74.1 (K), D75.1 (K), D78.1 (K)
- net at D73.2 (A): now also MX73.2 (ROW)
- net Row9: now reaches D38.1 (K)
- net Row9: now also D34.1 (K), D35.1 (K), D36.1 (K), D37.1 (K), D68.1 (K), D69.1 (K), D80.1 (K)
- net at D38.2 (A): now also MX38.2 (ROW)
- net Col3: now reaches MX3.1 (COL)
- net Col3: now also MX11.1 (COL), MX16.1 (COL), MX28.1 (COL), MX40.1 (COL), MX51.1 (COL), MX61.1 (COL), MX73.1 (COL), MX80.1 (COL), MX82.1 (COL), MX83.1 (COL), MX85.1 (COL)
- net at MX3.2 (ROW): now also D3.2 (A)
- net Row4: now reaches D81.1 (K)
- net Row4: now also D39.1 (K), D40.1 (K), D41.1 (K), D42.1 (K), D43.1 (K), D44.1 (K)
- net at D81.2 (A): now also MX81.2 (ROW)
- net at MX28.2 (ROW): now also D28.2 (A)
- net Row1: now reaches D7.1 (K)
- net Row1: now also D1.1 (K), D2.1 (K), D3.1 (K), D4.1 (K), D5.1 (K), D6.1 (K), D8.1 (K)
- net at D7.2 (A): now also MX7.2 (ROW)
- net Col4: now reaches MX41.1 (COL)
- net Col4: now also MX17.1 (COL), MX26.1 (COL), MX29.1 (COL), MX38.1 (COL), MX4.1 (COL), MX49.1 (COL), MX52.1 (COL), MX59.1 (COL), MX64.1 (COL), MX77.1 (COL), MX78.1 (COL)
- net at MX41.2 (ROW): now also D41.2 (A)
- net Row10: now reaches D47.1 (K)
- net Row10: now also D45.1 (K), D46.1 (K), D48.1 (K), D49.1 (K), D70.1 (K), D83.1 (K)
- net at D47.2 (A): now also MX47.2 (ROW)
- net Col8: now reaches MX9.1 (COL)
- net Col8: now also MX21.1 (COL), MX22.1 (COL), MX33.1 (COL), MX34.1 (COL), MX45.1 (COL), MX56.1 (COL), MX8.1 (COL)
- net at MX9.2 (ROW): now also D9.2 (A)
- net Col7: now reaches MX35.1 (COL)
- net Col7: now also MX10.1 (COL), MX20.1 (COL), MX23.1 (COL), MX32.1 (COL), MX44.1 (COL), MX46.1 (COL), MX55.1 (COL), MX7.1 (COL)
- net at MX35.2 (ROW): now also D35.2 (A)
- net Row6: now reaches D67.1 (K)
- net Row6: now also D22.1 (K), D23.1 (K), D24.1 (K), D25.1 (K), D26.1 (K), D60.1 (K), D61.1 (K), D66.1 (K), D76.1 (K), D77.1 (K), D82.1 (K), D86.1 (K)
- net at D67.2 (A): now also MX67.2 (ROW)
- net at D77.2 (A): now also MX77.2 (ROW)
- net at MX44.2 (ROW): now also D44.2 (A)
- net Col6: now reaches MX24.1 (COL)
- net Col6: now also MX12.1 (COL), MX19.1 (COL), MX31.1 (COL), MX36.1 (COL), MX43.1 (COL), MX47.1 (COL), MX54.1 (COL), MX57.1 (COL), MX6.1 (COL), MX62.1 (COL)
- net at MX24.2 (ROW): now also D24.2 (A)
- net at MX10.2 (ROW): now also D10.2 (A)
- net Row5: now reaches D53.1 (K)
- net Row5: now also D50.1 (K), D51.1 (K), D52.1 (K), D54.1 (K), D55.1 (K), D56.1 (K), D84.1 (K)
- net at D53.2 (A): now also MX53.2 (ROW)
- net at MX40.2 (ROW): now also D40.2 (A)
- net at MX46.2 (ROW): now also D46.2 (A)
- net at D45.2 (A): now also MX45.2 (ROW)
- net Col1: now reaches MX75.1 (COL)
- net Col1: now also MX1.1 (COL), MX14.1 (COL), MX67.1 (COL), MX69.1 (COL), MX70.1 (COL), MX71.1 (COL), MX76.1 (COL), MX79.1 (COL), MX81.1 (COL), MX84.1 (COL), SW1.S1
- net at MX75.2 (ROW): now also D75.2 (A)
- net at D2.2 (A): now also MX2.2 (ROW)
- net Row11: now reaches D58.1 (K)
- net Row11: now also D57.1 (K), D59.1 (K), D71.1 (K), D72.1 (K), D85.1 (K)
- net at D58.2 (A): now also MX58.2 (ROW)
- net at D55.2 (A): now also MX55.2 (ROW)
- net Col5: now reaches MX25.1 (COL)
- net Col5: now also MX13.1 (COL), MX18.1 (COL), MX30.1 (COL), MX37.1 (COL), MX42.1 (COL), MX48.1 (COL), MX5.1 (COL), MX53.1 (COL), MX58.1 (COL), MX63.1 (COL), MX86.1 (COL)
- net at MX25.2 (ROW): now also D25.2 (A)
- net Row7: now reaches D11.1 (K)
- net Row7: now also D10.1 (K), D12.1 (K), D13.1 (K), D64.1 (K), D65.1 (K), D87.1 (K), D9.1 (K)
- net at D11.2 (A): now also MX11.2 (ROW)
- net Col2: now reaches MX74.1 (COL)
- net Col2: now also MX15.1 (COL), MX2.1 (COL), MX27.1 (COL), MX39.1 (COL), MX50.1 (COL), MX60.1 (COL), MX65.1 (COL), MX66.1 (COL), MX68.1 (COL), MX72.1 (COL)
- net at MX74.2 (ROW): now also D74.2 (A)
- net at MX23.2 (ROW): now also D23.2 (A)
- net at MX26.2 (ROW): now also D26.2 (A)
- net Row2: now reaches D16.1 (K)
- net Row2: now also D14.1 (K), D15.1 (K), D17.1 (K), D18.1 (K), D19.1 (K), D20.1 (K), D21.1 (K)
- net at D16.2 (A): now also MX16.2 (ROW)
- net Row3: now reaches D27.1 (K)
- net Row3: now also D28.1 (K), D29.1 (K), D30.1 (K), D31.1 (K), D32.1 (K), D33.1 (K), D79.1 (K)
- net at D27.2 (A): now also MX27.2 (ROW)
- net at MX52.2 (ROW): now also D52.2 (A)
- net at D65.2 (A): now also MX65.2 (ROW)
- net at D22.2 (A): now also MX22.2 (ROW)
- net at D20.2 (A): now also MX20.2 (ROW)
- net at MX1.2 (ROW): now also D1.2 (A)
- net at MX4.2 (ROW): now also D4.2 (A)
- net at MX14.2 (ROW): now also D14.2 (A)
- net at MX17.2 (ROW): now also D17.2 (A)
- net at D39.2 (A): now also MX39.2 (ROW)
- net at D42.2 (A): now also MX42.2 (ROW)
- net at D18.2 (A): now also MX18.2 (ROW)
- net at MX29.2 (ROW): now also D29.2 (A)
- net at MX6.2 (ROW): now also D6.2 (A)
- net at MX70.2 (ROW): now also D70.2 (A)
- net at MX83.2 (ROW): now also D83.2 (A)
- net at MX82.2 (ROW): now also D82.2 (A)
- net at MX19.2 (ROW): now also D19.2 (A)
- net at MX62.2 (ROW): now also D62.2 (A)
- net at MX57.2 (ROW): now also D57.2 (A)
- net at D15.2 (A): now also MX15.2 (ROW)
- net at MX31.2 (ROW): now also D31.2 (A)
- net at D48.2 (A): now also MX48.2 (ROW)
- net at MX79.2 (ROW): now also D79.2 (A)
- net at D69.2 (A): now also MX69.2 (ROW)
- net at MX86.2 (ROW): now also D86.2 (A)
- net at D68.2 (A): now also MX68.2 (ROW)
- net at D50.2 (A): now also MX50.2 (ROW)
- net at MX5.2 (ROW): now also D5.2 (A)
- net at MX71.2 (ROW): now also D71.2 (A)
- net at D76.2 (A): now also MX76.2 (ROW)
- net at D43.2 (A): now also MX43.2 (ROW)
- net at D66.2 (A): now also MX66.2 (ROW)
- net at MX84.2 (ROW): now also D84.2 (A)
- net at MX56.2 (ROW): now also D56.2 (A)
- net at D36.2 (A): now also MX36.2 (ROW)
- net at MX80.2 (ROW): now also D80.2 (A)
- net at MX61.2 (ROW): now also D61.2 (A)
- net at MX49.2 (ROW): now also D49.2 (A)
- net at D63.2 (A): now also MX63.2 (ROW)
- net at MX59.2 (ROW): now also D59.2 (A)
- net at MX51.2 (ROW): now also D51.2 (A)
- net at MX54.2 (ROW): now also D54.2 (A)
- net at D85.2 (A): now also MX85.2 (ROW)
- net at MX8.2 (ROW): now also D8.2 (A)
- net at D13.2 (A): now also MX13.2 (ROW)
- net at D34.2 (A): now also MX34.2 (ROW)
- net at MX12.2 (ROW): now also D12.2 (A)
- net at MX60.2 (ROW): now also D60.2 (A)
- net at D37.2 (A): now also MX37.2 (ROW)
- net at MX32.2 (ROW): now also D32.2 (A)
- net at MX78.2 (ROW): now also D78.2 (A)
- net at D64.2 (A): now also MX64.2 (ROW)
- net at D30.2 (A): now also MX30.2 (ROW)
- net at MX72.2 (ROW): now also D72.2 (A)
- net at MX33.2 (ROW): now also D33.2 (A)
- net RRotA: now reaches SW1.A
- net RRotC: now reaches SW1.B
- net RRotB: now reaches SW1.C
- net RSw2: now reaches SW1.S2
- net RSw2: now also D87.2 (A)
- net at MX21.2 (ROW): now also D21.2 (A)
Other:
- moved on the sheet: D1, D10, D11, D12, D13, D14, D15, D16, D17, D18, D19, D2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

Commit message: routed minus rot and controller
Parts:
- removed D89: 1N4148W, Diode_SMD:D_SOD-123, symbol Device:D_Small
Connections:
- net RRotA is gone; now on net Col7: SW1.A
- net RRotB is gone; now on net RRotC: SW1.C
- net Col3: now also MX64.1 (COL); no longer MX11.1 (COL)
- net Col4: now also MX13.1 (COL); no longer MX64.1 (COL)
- net Col5: now also MX12.1 (COL); no longer MX13.1 (COL)
- net Col6: now also MX11.1 (COL); no longer MX12.1 (COL)
- net Col7: now also SW1.B
- net RRotC: now also D88.2 (A); no longer SW1.B
- net Row11: now also D88.1 (K)
Other:
- moved on the sheet: D1, D10, D11, D12, D13, D14, D15, D16, D17, D18, D19, D2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

Commit message: fully routed draft
Connections:
- net Col1: now also U1.17 (P1.15)
- net Col2: now also U1.16 (P1.13)
- net Col3: now also U1.31 (P1.01)
- net Col4: now also U1.7 (P0.22)
- net Col5: now also U1.8 (P0.24)
- net Col6: now also U1.9 (P1.00)
- net Col7: now also U1.33 (P1.07); no longer SW1.B
- net Col8: now also SW1.B, U1.32 (P1.02)
- net Row1: now also U1.13 (NFC1/P0.09)
- net Row11: now also U1.5 (P0.17)
- net Row12: now also U1.6 (P0.20)
- net Row2: now also U1.14 (NFC2/P0.10)
- net Row3: now also U1.15 (P1.11)
- net Row4: now also U1.10 (P0.11)
- net Row5: now also U1.11 (P1.04)
- net Row6: now also U1.12 (P1.06); no longer D22.1 (K), D23.1 (K), D24.1 (K), D25.1 (K), D26.1 (K), D66.1 (K), D67.1 (K), D82.1 (K)
- net Row7: now also U1.18 (AIN0/P0.02)
- net Row9: now also U1.20 (AIN7/P0.31)
- net Row8: now reaches U1.19 (AIN5/P0.29)
- net Row8: now also D22.1 (K), D23.1 (K), D24.1 (K), D25.1 (K), D26.1 (K), D66.1 (K), D67.1 (K), D82.1 (K)
Other:
- moved on the sheet: D1, D10, D11, D12, D13, D14, D15, D16, D17, D18, D19, D2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

Commit message: most diodes rerouted to back
Connections:
- net Col4: now also U1.6 (P0.20); no longer U1.7 (P0.22)
- net Col5: now also U1.5 (P0.17); no longer U1.8 (P0.24)
- net Col6: now also U1.1 (TX0/P0.06); no longer U1.9 (P1.00)
- net Col7: now also U1.32 (P1.02); no longer U1.33 (P1.07)
- net Col8: now also U1.33 (P1.07); no longer U1.32 (P1.02)
- net Row10: now also U1.9 (P1.00)
- net Row11: now also U1.8 (P0.24); no longer U1.5 (P0.17)
- net Row12: now also U1.7 (P0.22); no longer U1.6 (P0.20)
Changed lines of the file:
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@@
 	)
 	(label "Col7"
-		(at 90.17 154.94 180)
+		(at 90.17 158.75 180)
 		(effects
 			(font
@@
 	)
 	(label "Row11"
-		(at 120.65 172.72 270)
+		(at 113.03 172.72 270)
 		(effects
 			(font
@@
 	)
 	(label "Col4"
-		(at 115.57 172.72 270)
+		(at 118.11 172.72 270)
 		(effects
 			(font
@@
 	)
 	(label "Col8"
-		(at 90.17 158.75 180)
+		(at 90.17 154.94 180)
 		(effects
 			(font
@@
 	)
 	(label "Col5"
-		(at 113.03 172.72 270)
+		(at 120.65 172.72 270)
 		(effects
 			(font
@@
 	)
 	(label "Row10"
-		(at 130.81 173.99 270)
+		(at 110.49 172.72 270)
 		(effects
 			(font
@@
 	)
 	(label "Row12"
-		(at 118.11 172.72 270)
+		(at 115.57 172.72 270)
 		(effects
 			(font
@@
 	)
 	(label "Col6"
-		(at 110.49 172.72 270)
-		(effects
-			(font
+		(at 130.81 172.72 270)
+		(effects
+			(font

Commit message: pcbs ordered july 13th 2025
Connections:
- net Col5: now also U1.32 (P1.02); no longer U1.5 (P0.17)
- net Col7: now also U1.5 (P0.17); no longer U1.32 (P1.02)
Changed lines of the file:
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@@
 	)
 	(label "Col7"
-		(at 90.17 158.75 180)
+		(at 120.65 172.72 270)
 		(effects
 			(font
@@
 	)
 	(label "Col5"
-		(at 120.65 172.72 270)
+		(at 90.17 158.75 180)
 		(effects
 			(font
